Commit message: joint names changed to motor_down and motor_up

File: urdf/gripper_6.urdf.xacro (robot description, xacro)
@@ -95,5 +95,5 @@
     </link>
 	<!-- continuous motor up m1-->
-	<joint name="${prefix}gripper_motorup_joint" type="continuous">
+	<joint name="${prefix}gripper_motor_up_joint" type="continuous">
       <origin xyz="0 0.159 0.126" rpy="0 0 0"/>
       <parent link="${prefix}gripper_base_link"/>
@@ -123,5 +123,5 @@
     </link>
     <!-- continuous motor down m2-->
-	<joint name="${prefix}gripper_motordown_joint" type="continuous">
+	<joint name="${prefix}gripper_motor_down_joint" type="continuous">
       <origin xyz="0 0.159 0.287" rpy="0 0 0"/>
       <parent link="${prefix}gripper_base_link"/>
@@ -185,5 +185,5 @@
       <parent link="${prefix}gripper_prismatic_link"/>
       <child link="${prefix}gripper_revolute_link"/>
-      <limit lower="-0.35" upper="0.35" effort="0" velocity="${DEG2RAD * 330}"/>
+      <limit lower="0.0" upper="0.79" effort="0" velocity="${DEG2RAD * 330}"/>
       <axis xyz="-1 0 0"/>
     </joint>

Commit message: axis of traslation inverted

File: urdf/gripper_6.urdf.xacro (robot description, xacro)
@@ -98,10 +98,10 @@
       <origin xyz="0 0.159 0.126" rpy="0 0 0"/>
       <parent link="${prefix}gripper_base_link"/>
-      <child link="${prefix}gripper_motorup_link"/>
+      <child link="${prefix}gripper_motor_up_link"/>
       <limit effort="100.0" velocity="0.005"/>
       <axis xyz="0 1 0"/>
     </joint>
     <!-- ROS base_link to gripper motor up 1 coordinate system transform -->
-    <link name="${prefix}gripper_motorup_link">
+    <link name="${prefix}gripper_motor_up_link">
      <inertial>
       <origin rpy="0 0 0" xyz="0.0 0.0 0.0"/>
@@ -126,10 +126,10 @@
       <origin xyz="0 0.159 0.287" rpy="0 0 0"/>
       <parent link="${prefix}gripper_base_link"/>
-      <child link="${prefix}gripper_motordown_link"/>
+      <child link="${prefix}gripper_motor_down_link"/>
       <limit effort="100.0" velocity="0.005"/>
       <axis xyz="0 1 0"/>
     </joint>
     <!-- ROS base_link to gripper motor up 1 coordinate system transform -->
-    <link name="${prefix}gripper_motordown_link">
+    <link name="${prefix}gripper_motor_down_link">
      <inertial>
       <origin rpy="0 0 0" xyz="0.0 0.0 0.0"/>
@@ -156,5 +156,5 @@
       <child link="${prefix}gripper_prismatic_link"/>
       <limit effort="100.0" velocity="0.5" lower="-0.105" upper="0.105"/>
-      <axis xyz="0 1 0"/>
+      <axis xyz="0 -1 0"/>
     </joint>
     <!-- ROS base_link to gripper coordinate system transform -->
@@ -262,6 +262,6 @@
       </collision>
     </link>
-   <xacro:motor_simple_transmission name="${prefix}gripper_motorup_joint"/>
-   <xacro:motor_simple_transmission name="${prefix}gripper_motordown_joint"/>
+   <xacro:motor_simple_transmission name="${prefix}gripper_motor_up_joint"/>
+   <xacro:motor_simple_transmission name="${prefix}gripper_motor_down_joint"/>
    <xacro:simple_transmission name="${prefix}gripper_revolute_joint"/>
    <xacro:simple_transmission name="${prefix}gripper_prismatic_joint"/>

Commit message: finger origin changed

File: urdf/gripper_6.urdf.xacro (robot description, xacro)
@@ -152,8 +152,8 @@
    <!-- prismatic -->
 	<joint name="${prefix}gripper_prismatic_joint" type="prismatic">
-      <origin xyz="0.0 0.0 0.0" rpy="0 0 0"/>
+      <origin xyz="0.0 0.105 0.0" rpy="0 0 0"/>
       <parent link="${prefix}gripper_base_link"/>
       <child link="${prefix}gripper_prismatic_link"/>
-      <limit effort="100.0" velocity="0.5" lower="-0.105" upper="0.105"/>
+      <limit effort="100.0" velocity="0.5" lower="-0.210" upper="0.0"/>
       <axis xyz="0 -1 0"/>
     </joint>

Commit message: added marker link frame to calibrate cameras

File: urdf/gripper_6.urdf.xacro (robot description, xacro)
@@ -68,4 +68,19 @@
       </collision>
     </link>
+    <!-- QR marker -->
+    <!-- 160 de ancho 185 de alto respecto a tool0 o gripper_base_link-->
+	<joint name="${prefix}gripper_marker_joint" type="fixed">
+      <origin xyz="0.0 -0.160 0.2065" rpy="0 0 ${-PI}"/>
+      <parent link="${prefix}gripper_base_link"/>
+      <child link="${prefix}gripper_marker_fixed_link"/>
+    </joint>
+    <!-- QR marker -->
+    <link name="${prefix}gripper_marker_fixed_link">
+     <inertial>
+      <origin rpy="0 0 0" xyz="0.0 0.0 0.0"/>
+      <mass value="0.1"/>
+      <inertia ixx="0.001" ixy="0.0" ixz="0.0" iyy="0.001" iyz="0.0" izz="0.001"/>
+    </inertial>
+    </link>
     <!-- finger fixed -->
 	<joint name="${prefix}gripper_finger_fixed_joint" type="fixed">
